Commit message: Fix inverse kinematics

File: torch_robotics/data/urdf/robots/franka_description/robots/panda_arm_hand.urdf (robot description, URDF)
Before this commit: robot panda, 12 links, 11 joints
Links:
- added link ee_link; collision box size=0.01 0.01 0.01
Joints:
- added joint ee_fixed_joint: type fixed, parent panda_hand, child ee_link, origin xyz=0.0 0. 0.1 rpy=0.0 0.0 -1.57
