Commit message: Integrate grasping in isaac

File: torch_robotics/data/urdf/robots/franka_description/robots/panda_arm_no_gripper_grasped_object.urdf (robot description, URDF)
Before this commit: robot panda, 12 links, 11 joints
Joints:
- joint grasped_object_fixed_joint: origin xyz=0.0 0.0 0.05 rpy=1.5707965 0.0 0.0 -> xyz=0.0 0.0 0.11 rpy=3.1415927 -1.5707964 0.0; parent ee_link -> panda_hand
