Commit message: Forward kinematics with torchkin and get gradient of sdf

File: torch_robotics/data/urdf/robots/franka_description/robots/hand.xacro (robot description, xacro)
@@ -20,9 +20,4 @@
         </geometry>
       </collision>
-      <inertial>
-        <origin rpy="0 0 0" xyz="0 0 0" />
-        <mass value="0.5583304799"/>
-        <inertia ixx="0.0023394448" ixy="0.0" ixz="0.0" iyy="0.0005782786" iyz="0" izz="0.0021310296"/>
-      </inertial>
     </link>
     <link name="${ns}_leftfinger">
@@ -37,9 +32,4 @@
         </geometry>
       </collision>
-      <inertial>
-        <origin rpy="0 0 0" xyz="0 0 0" />
-        <mass value="0.0140552232"/>
-        <inertia ixx="4.20413082650939E-06" ixy="0.0" ixz="0.0" iyy="3.90263687466755E-06" iyz="0" izz="1.33474964199095E-06"/>
-      </inertial>
     </link>
     <link name="${ns}_rightfinger">
@@ -56,9 +46,4 @@
         </geometry>
       </collision>
-      <inertial>
-        <origin rpy="0 0 0" xyz="0 0 0" />
-        <mass value="0.0140552232"/>
-        <inertia ixx="4.20413082650939E-06" ixy="0.0" ixz="0.0" iyy="3.90263687466755E-06" iyz="0" izz="1.33474964199095E-06"/>
-      </inertial>
     </link>
     <joint name="${ns}_finger_joint1" type="prismatic">

File: torch_robotics/data/urdf/robots/franka_description/robots/panda_arm.urdf (robot description, URDF)
Before this commit: robot panda, 9 links, 8 joints
Links:
- link panda_link0: mass 2.8142028896 -> None
- link panda_link1: mass 2.3599995791 -> None
- link panda_link2: mass 2.379518833 -> None
- link panda_link3: mass 2.6498823337 -> None
- link panda_link4: mass 2.6948018744 -> None
- link panda_link5: mass 2.9812816864 -> None
- link panda_link6: mass 1.1285806309 -> None
- link panda_link7: mass 0.4052912465 -> None

File: torch_robotics/data/urdf/robots/franka_description/robots/panda_arm.urdf.xacro (robot description, xacro)
@@ -1,5 +1,5 @@
-<?xml version="1.0" encoding="utf-8"?>
+<?xml version='1.0' encoding='utf-8'?>
 <robot xmlns:xacro="http://www.ros.org/wiki/xacro" name="panda">
-  <xacro:include filename="$(find franka_description)/robots/panda_arm.xacro"/>
+  <xacro:include filename="$(find franka_description)/robots/panda_arm.xacro" />
   <xacro:panda_arm />
 </robot>

File: torch_robotics/data/urdf/robots/franka_description/robots/panda_arm.xacro (robot description, xacro)
@@ -20,9 +20,4 @@
         </geometry>
       </collision>
-      <inertial>
-        <origin rpy="0 0 0" xyz="0 0 0"/>
-        <mass value="2.8142028896"/>
-        <inertia ixx="0.0129886979" ixy="0.0" ixz="0.0" iyy="0.0165355284" iyz="0" izz="0.0203311636"/>
-      </inertial>
     </link>
     <link name="${arm_id}_link1">
@@ -37,9 +32,4 @@
         </geometry>
       </collision>
-      <inertial>
-        <origin rpy="0 0 0" xyz="0 0 0" />
-        <mass value="2.3599995791"/>
-        <inertia ixx="0.0186863903" ixy="0.0" ixz="0.0" iyy="0.0143789874" iyz="0" izz="0.00906812"/>
-      </inertial>
     </link>
     <joint name="${arm_id}_joint1" type="revolute">
@@ -62,9 +52,4 @@
         </geometry>
       </collision>
-      <inertial>
-        <origin rpy="0 0 0" xyz="0 0 0" />
-        <mass value="2.379518833" />
-        <inertia ixx="0.0190388734" ixy="0.0" ixz="0.0" iyy="0.0091429124" iyz="0" izz="0.014697537"/>
-      </inertial>
     </link>
     <joint name="${arm_id}_joint2" type="revolute">
@@ -87,9 +72,4 @@
         </geometry>
       </collision>
-      <inertial>
-        <origin rpy="0 0 0" xyz="0 0 0" />
-        <mass value="2.6498823337"/>
-        <inertia ixx="0.0129300178" ixy="0.0" ixz="0.0" iyy="0.0150242121" iyz="0" izz="0.0142734598"/>
-      </inertial>
     </link>
     <joint name="${arm_id}_joint3" type="revolute">
@@ -112,9 +92,4 @@
         </geometry>
       </collision>
-      <inertial>
-        <origin rpy="0 0 0" xyz="0 0 0" />
-        <mass value="2.6948018744"/>
-        <inertia ixx="0.0133874611" ixy="0.0" ixz="0.0" iyy="0.014514325" iyz="0" izz="0.0155175551"/>
-      </inertial>
     </link>
     <joint name="${arm_id}_joint4" type="revolute">
@@ -137,9 +112,4 @@
         </geometry>
       </collision>
-      <inertial>
-        <origin rpy="0 0 0" xyz="0 0 0" />
-        <mass value="2.9812816864"/>
-        <inertia ixx="0.0325565705" ixy="0.0" ixz="0.0" iyy="0.0270660472" iyz="0" izz="0.0115023375"/>
-      </inertial>
     </link>
     <joint name="${arm_id}_joint5" type="revolute">
@@ -162,9 +132,4 @@
         </geometry>
       </collision>
-      <inertial>
-        <origin rpy="0 0 0" xyz="0 0 0" />
-        <mass value="1.1285806309"/>
-        <inertia ixx="0.0026052565" ixy="0.0" ixz="0.0" iyy="0.0039897229" iyz="0" izz="0.0047048591"/>
-      </inertial>
     </link>
     <joint name="${arm_id}_joint6" type="revolute">
@@ -187,9 +152,4 @@
         </geometry>
       </collision>
-      <inertial>
-        <origin rpy="0 0 0" xyz="0 0 0" />
-        <mass value="0.4052912465"/>
-        <inertia ixx="0.0006316592" ixy="0.0" ixz="0.0" iyy="0.0006319639" iyz="0" izz="0.0010607721"/>
-      </inertial>
     </link>
     <joint name="${arm_id}_joint7" type="revolute">

File: torch_robotics/data/urdf/robots/franka_description/robots/panda_arm_hand.urdf (robot description, URDF)
Before this commit: robot panda, 13 links, 12 joints
Links:
- removed link ee_link
- added link tool_link
- link panda_hand: mass 0.5583304799 -> None
- link panda_leftfinger: mass 0.0140552232 -> None
- link panda_link0: mass 2.8142028896 -> None
- link panda_link1: mass 2.3599995791 -> None
- link panda_link2: mass 2.379518833 -> None
- link panda_link3: mass 2.6498823337 -> None
- link panda_link4: mass 2.6948018744 -> None
- link panda_link5: mass 2.9812816864 -> None
- link panda_link6: mass 1.1285806309 -> None
- link panda_link7: mass 0.4052912465 -> None
- link panda_rightfinger: mass 0.0140552232 -> None
Joints:
- removed joint ee_fixed_joint
- added joint tool_joint: type fixed, parent panda_link8, child tool_link, origin xyz=0.0 0 0.1 rpy=0 0 2.35619449019, axis 0 0 1

File: torch_robotics/data/urdf/robots/franka_description/robots/panda_arm_no_gripper_collision_model.urdf (robot description, URDF)
Before this commit: robot panda, 55 links, 54 joints
Links:
- added link panda_hand_12
- added link panda_hand_13
- added link panda_hand_14
- added link panda_hand_15
- added link panda_hand_16
- added link panda_hand_17
Joints:
- added joint joint_panda_hand_sphere_12: type fixed, parent panda_hand, child panda_hand_12, origin xyz=0.0 -0.075 0.05 rpy=0 0 0
- added joint joint_panda_hand_sphere_13: type fixed, parent panda_hand, child panda_hand_13, origin xyz=0.0 -0.045 0.05 rpy=0 0 0
- added joint joint_panda_hand_sphere_14: type fixed, parent panda_hand, child panda_hand_14, origin xyz=0.0 -0.015 0.05 rpy=0 0 0
- added joint joint_panda_hand_sphere_15: type fixed, parent panda_hand, child panda_hand_15, origin xyz=0.0 0.015 0.05 rpy=0 0 0
- added joint joint_panda_hand_sphere_16: type fixed, parent panda_hand, child panda_hand_16, origin xyz=0.0 0.045 0.05 rpy=0 0 0
- added joint joint_panda_hand_sphere_17: type fixed, parent panda_hand, child panda_hand_17, origin xyz=0.0 0.075 0.05 rpy=0 0 0
- joint joint_panda_hand_sphere_1: origin xyz=0.0 -0.015 0.01 rpy=0 0 0 -> xyz=0.0 -0.045 0.01 rpy=0 0 0
- joint joint_panda_hand_sphere_10: origin xyz=0.0 0.015 0.05 rpy=0 0 0 -> xyz=0.0 0.045 0.03 rpy=0 0 0
- joint joint_panda_hand_sphere_11: origin xyz=0.0 0.075 0.05 rpy=0 0 0 -> xyz=0.0 0.075 0.03 rpy=0 0 0
- joint joint_panda_hand_sphere_2: origin xyz=0.0 0.015 0.01 rpy=0 0 0 -> xyz=0.0 -0.015 0.01 rpy=0 0 0
- joint joint_panda_hand_sphere_3: origin xyz=0.0 0.075 0.01 rpy=0 0 0 -> xyz=0.0 0.015 0.01 rpy=0 0 0
- joint joint_panda_hand_sphere_4: origin xyz=0.0 -0.075 0.03 rpy=0 0 0 -> xyz=0.0 0.045 0.01 rpy=0 0 0
- joint joint_panda_hand_sphere_5: origin xyz=0.0 -0.015 0.03 rpy=0 0 0 -> xyz=0.0 0.075 0.01 rpy=0 0 0
- joint joint_panda_hand_sphere_6: origin xyz=0.0 0.015 0.03 rpy=0 0 0 -> xyz=0.0 -0.075 0.03 rpy=0 0 0
- joint joint_panda_hand_sphere_7: origin xyz=0.0 0.075 0.03 rpy=0 0 0 -> xyz=0.0 -0.045 0.03 rpy=0 0 0
- joint joint_panda_hand_sphere_8: origin xyz=0.0 -0.075 0.05 rpy=0 0 0 -> xyz=0.0 -0.015 0.03 rpy=0 0 0
- joint joint_panda_hand_sphere_9: origin xyz=0.0 -0.015 0.05 rpy=0 0 0 -> xyz=0.0 0.015 0.03 rpy=0 0 0
