Commit message: Fix grasped object urdf

File: torch_robotics/data/urdf/robots/franka_description/robots/panda_arm_hand_fixed_gripper_collision_model_grasped_object.urdf (robot description, URDF)
Before this commit: robot panda, 78 links, 77 joints
Links:
- link link_GraspedObjectBox: geometry collision box size=0.05 0.05 0.1; visual box size=0.05 0.05 0.1
Joints:
- joint joint_fixed_GraspedObjectBox: origin xyz=0.0 0.0 0.11 rpy=3.1415927 -1.5707964 0.0 -> xyz=0.0 0.0 0.11 rpy=0.0 -1.5704511 0.0
- joint joint_fixed_GraspedObjectBox_point_0: origin xyz=0.025 0.025 -0.075 rpy=0 0 0 -> xyz=0.025 0.025 -0.05 rpy=0 0 0; parent panda_hand -> link_GraspedObjectBox
- joint joint_fixed_GraspedObjectBox_point_1: origin xyz=0.025 -0.025 -0.075 rpy=0 0 0 -> xyz=0.025 -0.025 -0.05 rpy=0 0 0; parent panda_hand -> link_GraspedObjectBox
- joint joint_fixed_GraspedObjectBox_point_10: parent panda_hand -> link_GraspedObjectBox
- joint joint_fixed_GraspedObjectBox_point_11: parent panda_hand -> link_GraspedObjectBox
- joint joint_fixed_GraspedObjectBox_point_12: origin xyz=0.0 0.0 0.075 rpy=0 0 0 -> xyz=0.0 0.0 0.05 rpy=0 0 0; parent panda_hand -> link_GraspedObjectBox
- joint joint_fixed_GraspedObjectBox_point_13: origin xyz=0.0 0.0 -0.075 rpy=0 0 0 -> xyz=0.0 0.0 -0.05 rpy=0 0 0; parent panda_hand -> link_GraspedObjectBox
- joint joint_fixed_GraspedObjectBox_point_2: origin xyz=-0.025 -0.025 -0.075 rpy=0 0 0 -> xyz=-0.025 -0.025 -0.05 rpy=0 0 0; parent panda_hand -> link_GraspedObjectBox
- joint joint_fixed_GraspedObjectBox_point_3: origin xyz=-0.025 0.025 -0.075 rpy=0 0 0 -> xyz=-0.025 0.025 -0.05 rpy=0 0 0; parent panda_hand -> link_GraspedObjectBox
- joint joint_fixed_GraspedObjectBox_point_4: origin xyz=0.025 0.025 0.075 rpy=0 0 0 -> xyz=0.025 0.025 0.05 rpy=0 0 0; parent panda_hand -> link_GraspedObjectBox
- joint joint_fixed_GraspedObjectBox_point_5: origin xyz=0.025 -0.025 0.075 rpy=0 0 0 -> xyz=0.025 -0.025 0.05 rpy=0 0 0; parent panda_hand -> link_GraspedObjectBox
- joint joint_fixed_GraspedObjectBox_point_6: origin xyz=-0.025 -0.025 0.075 rpy=0 0 0 -> xyz=-0.025 -0.025 0.05 rpy=0 0 0; parent panda_hand -> link_GraspedObjectBox
- joint joint_fixed_GraspedObjectBox_point_7: origin xyz=-0.025 0.025 0.075 rpy=0 0 0 -> xyz=-0.025 0.025 0.05 rpy=0 0 0; parent panda_hand -> link_GraspedObjectBox
- joint joint_fixed_GraspedObjectBox_point_8: parent panda_hand -> link_GraspedObjectBox
- joint joint_fixed_GraspedObjectBox_point_9: parent panda_hand -> link_GraspedObjectBox
- joint panda_finger_joint1: origin xyz=0.0 0.0 0.0584 rpy=0.0 0.0 0.0 -> xyz=0.0 0.04 0.0584 rpy=0.0 0.0 0.0; type prismatic -> fixed
- joint panda_finger_joint2: origin xyz=0.0 0.0 0.0584 rpy=0.0 0.0 0.0 -> xyz=0.0 -0.04 0.0584 rpy=0.0 0.0 0.0; type prismatic -> fixed

File: torch_robotics/data/urdf/robots/franka_description/robots/panda_arm_hand_fixed_gripper_grasped_object_collision_model.urdf (robot description, URDF)
Before this commit: robot panda, 76 links, 75 joints
Links:
- removed link ee_link
- added link panda_leftfinger; collision mesh filename=package://franka_description/meshes/collision/finger.stl; visual mesh filename=package://franka_description/meshes/visual/finger.dae
- added link panda_rightfinger; collision mesh filename=package://franka_description/meshes/collision/finger.stl; visual mesh filename=package://franka_description/meshes/visual/finger.dae
- added link tool_link
- link link_GraspedObjectBox: geometry collision box size=0.05 0.05 0.1; visual box size=0.05 0.05 0.1
- link panda_hand: mass 0.5583304799 -> None
- link panda_hand_0: geometry 
- link panda_hand_1: geometry 
- link panda_hand_10: geometry 
- link panda_hand_11: geometry 
- link panda_hand_12: geometry 
- link panda_hand_13: geometry 
- link panda_hand_14: geometry 
- link panda_hand_15: geometry 
- link panda_hand_16: geometry 
- link panda_hand_17: geometry 
- link panda_hand_2: geometry 
- link panda_hand_3: geometry 
- link panda_hand_4: geometry 
- link panda_hand_5: geometry 
- link panda_hand_6: geometry 
- link panda_hand_7: geometry 
- link panda_hand_8: geometry 
- link panda_hand_9: geometry 
- link panda_link0: mass 2.8142028896 -> None
- link panda_link1: mass 2.3599995791 -> None
- link panda_link2: mass 2.379518833 -> None
- link panda_link2_0: geometry 
- link panda_link2_1: geometry 
- link panda_link2_2: geometry 
- link panda_link2_3: geometry 
- link panda_link3: mass 2.6498823337 -> None
- link panda_link3_0: geometry 
- link panda_link3_1: geometry 
- link panda_link3_2: geometry 
- link panda_link3_3: geometry 
- link panda_link4: mass 2.6948018744 -> None
- link panda_link4_0: geometry 
- link panda_link4_1: geometry 
- link panda_link4_2: geometry 
- link panda_link4_3: geometry 
- link panda_link5: mass 2.9812816864 -> None
- link panda_link5_0: geometry 
- link panda_link5_1: geometry 
- link panda_link5_10: geometry 
- link panda_link5_11: geometry 
- link panda_link5_2: geometry 
- link panda_link5_3: geometry 
- link panda_link5_4: geometry 
- link panda_link5_5: geometry 
- link panda_link5_6: geometry 
- link panda_link5_7: geometry 
- link panda_link5_8: geometry 
- link panda_link5_9: geometry 
- link panda_link6: mass 1.1285806309 -> None
- link panda_link6_0: geometry 
- link panda_link6_1: geometry 
- link panda_link6_2: geometry 
- link panda_link7: mass 0.4052912465 -> None
- link panda_link7_0: geometry 
- link panda_link7_1: geometry 
- link panda_link7_2: geometry 
- link panda_link7_3: geometry 
- link panda_link7_4: geometry 
Joints:
- removed joint ee_fixed_joint
- added joint panda_finger_joint1: type fixed, parent panda_hand, child panda_leftfinger, origin xyz=0.0 0.04 0.0584 rpy=0.0 0.0 0.0, axis 0.0 1.0 0.0, limit lower=0.0 upper=0.04 effort=20.0 velocity=0.2
- added joint panda_finger_joint2: type fixed, parent panda_hand, child panda_rightfinger, origin xyz=0.0 -0.04 0.0584 rpy=0.0 0.0 0.0, axis 0.0 -1.0 0.0, limit lower=0.0 upper=0.04 effort=20.0 velocity=0.2, mimic joint=panda_finger_joint1
- added joint tool_joint: type fixed, parent panda_link8, child tool_link, origin xyz=0.0 0.0 0.1 rpy=0.0 0.0 2.35619449019, axis 0.0 0.0 1.0
- joint joint_fixed_GraspedObjectBox: origin xyz=0.0 0.0 0.11 rpy=3.1415927 -1.5707964 0.0 -> xyz=0.0 0.0 0.11 rpy=0.0 -1.5704511 0.0
- joint joint_fixed_GraspedObjectBox_point_0: origin xyz=0.025 0.025 -0.075 rpy=0 0 0 -> xyz=0.025 0.025 -0.05 rpy=0.0 0.0 0.0; parent panda_hand -> link_GraspedObjectBox
- joint joint_fixed_GraspedObjectBox_point_1: origin xyz=0.025 -0.025 -0.075 rpy=0 0 0 -> xyz=0.025 -0.025 -0.05 rpy=0.0 0.0 0.0; parent panda_hand -> link_GraspedObjectBox
- joint joint_fixed_GraspedObjectBox_point_10: origin xyz=-0.025 0.0 0.0 rpy=0 0 0 -> xyz=-0.025 0.0 0.0 rpy=0.0 0.0 0.0; parent panda_hand -> link_GraspedObjectBox
- joint joint_fixed_GraspedObjectBox_point_11: origin xyz=0.0 0.025 0.0 rpy=0 0 0 -> xyz=0.0 0.025 0.0 rpy=0.0 0.0 0.0; parent panda_hand -> link_GraspedObjectBox
- joint joint_fixed_GraspedObjectBox_point_12: origin xyz=0.0 0.0 0.075 rpy=0 0 0 -> xyz=0.0 0.0 0.05 rpy=0.0 0.0 0.0; parent panda_hand -> link_GraspedObjectBox
- joint joint_fixed_GraspedObjectBox_point_13: origin xyz=0.0 0.0 -0.075 rpy=0 0 0 -> xyz=0.0 0.0 -0.05 rpy=0.0 0.0 0.0; parent panda_hand -> link_GraspedObjectBox
- joint joint_fixed_GraspedObjectBox_point_2: origin xyz=-0.025 -0.025 -0.075 rpy=0 0 0 -> xyz=-0.025 -0.025 -0.05 rpy=0.0 0.0 0.0; parent panda_hand -> link_GraspedObjectBox
- joint joint_fixed_GraspedObjectBox_point_3: origin xyz=-0.025 0.025 -0.075 rpy=0 0 0 -> xyz=-0.025 0.025 -0.05 rpy=0.0 0.0 0.0; parent panda_hand -> link_GraspedObjectBox
- joint joint_fixed_GraspedObjectBox_point_4: origin xyz=0.025 0.025 0.075 rpy=0 0 0 -> xyz=0.025 0.025 0.05 rpy=0.0 0.0 0.0; parent panda_hand -> link_GraspedObjectBox
- joint joint_fixed_GraspedObjectBox_point_5: origin xyz=0.025 -0.025 0.075 rpy=0 0 0 -> xyz=0.025 -0.025 0.05 rpy=0.0 0.0 0.0; parent panda_hand -> link_GraspedObjectBox
- joint joint_fixed_GraspedObjectBox_point_6: origin xyz=-0.025 -0.025 0.075 rpy=0 0 0 -> xyz=-0.025 -0.025 0.05 rpy=0.0 0.0 0.0; parent panda_hand -> link_GraspedObjectBox
- joint joint_fixed_GraspedObjectBox_point_7: origin xyz=-0.025 0.025 0.075 rpy=0 0 0 -> xyz=-0.025 0.025 0.05 rpy=0.0 0.0 0.0; parent panda_hand -> link_GraspedObjectBox
- joint joint_fixed_GraspedObjectBox_point_8: origin xyz=0.025 0.0 0.0 rpy=0 0 0 -> xyz=0.025 0.0 0.0 rpy=0.0 0.0 0.0; parent panda_hand -> link_GraspedObjectBox
- joint joint_fixed_GraspedObjectBox_point_9: origin xyz=0.0 -0.025 0.0 rpy=0 0 0 -> xyz=0.0 -0.025 0.0 rpy=0.0 0.0 0.0; parent panda_hand -> link_GraspedObjectBox
- joint joint_panda_hand_sphere_0: origin xyz=0.0 -0.075 0.01 rpy=0.0 0.0 0.0 -> xyz=0.0 -0.075 0.01 rpy=0 0 0
- joint joint_panda_hand_sphere_1: origin xyz=0.0 -0.045 0.01 rpy=0.0 0.0 0.0 -> xyz=0.0 -0.045 0.01 rpy=0 0 0
- joint joint_panda_hand_sphere_10: origin xyz=0.0 0.045 0.03 rpy=0.0 0.0 0.0 -> xyz=0.0 0.045 0.03 rpy=0 0 0
- joint joint_panda_hand_sphere_11: origin xyz=0.0 0.075 0.03 rpy=0.0 0.0 0.0 -> xyz=0.0 0.075 0.03 rpy=0 0 0
- joint joint_panda_hand_sphere_12: origin xyz=0.0 -0.075 0.05 rpy=0.0 0.0 0.0 -> xyz=0.0 -0.075 0.05 rpy=0 0 0
- joint joint_panda_hand_sphere_13: origin xyz=0.0 -0.045 0.05 rpy=0.0 0.0 0.0 -> xyz=0.0 -0.045 0.05 rpy=0 0 0
- joint joint_panda_hand_sphere_14: origin xyz=0.0 -0.015 0.05 rpy=0.0 0.0 0.0 -> xyz=0.0 -0.015 0.05 rpy=0 0 0
- joint joint_panda_hand_sphere_15: origin xyz=0.0 0.015 0.05 rpy=0.0 0.0 0.0 -> xyz=0.0 0.015 0.05 rpy=0 0 0
- joint joint_panda_hand_sphere_16: origin xyz=0.0 0.045 0.05 rpy=0.0 0.0 0.0 -> xyz=0.0 0.045 0.05 rpy=0 0 0
- joint joint_panda_hand_sphere_17: origin xyz=0.0 0.075 0.05 rpy=0.0 0.0 0.0 -> xyz=0.0 0.075 0.05 rpy=0 0 0
- joint joint_panda_hand_sphere_2: origin xyz=0.0 -0.015 0.01 rpy=0.0 0.0 0.0 -> xyz=0.0 -0.015 0.01 rpy=0 0 0
- joint joint_panda_hand_sphere_3: origin xyz=0.0 0.015 0.01 rpy=0.0 0.0 0.0 -> xyz=0.0 0.015 0.01 rpy=0 0 0
- joint joint_panda_hand_sphere_4: origin xyz=0.0 0.045 0.01 rpy=0.0 0.0 0.0 -> xyz=0.0 0.045 0.01 rpy=0 0 0
- joint joint_panda_hand_sphere_5: origin xyz=0.0 0.075 0.01 rpy=0.0 0.0 0.0 -> xyz=0.0 0.075 0.01 rpy=0 0 0
- joint joint_panda_hand_sphere_6: origin xyz=0.0 -0.075 0.03 rpy=0.0 0.0 0.0 -> xyz=0.0 -0.075 0.03 rpy=0 0 0
- joint joint_panda_hand_sphere_7: origin xyz=0.0 -0.045 0.03 rpy=0.0 0.0 0.0 -> xyz=0.0 -0.045 0.03 rpy=0 0 0
- joint joint_panda_hand_sphere_8: origin xyz=0.0 -0.015 0.03 rpy=0.0 0.0 0.0 -> xyz=0.0 -0.015 0.03 rpy=0 0 0
- joint joint_panda_hand_sphere_9: origin xyz=0.0 0.015 0.03 rpy=0.0 0.0 0.0 -> xyz=0.0 0.015 0.03 rpy=0 0 0
- joint joint_panda_link2_sphere_0: origin xyz=0.0 0.0 0.03 rpy=0.0 0.0 0.0 -> xyz=0.0 0.0 0.03 rpy=0 0 0
- joint joint_panda_link2_sphere_1: origin xyz=0.0 0.0 0.08 rpy=0.0 0.0 0.0 -> xyz=0.0 0.0 0.08 rpy=0 0 0
- joint joint_panda_link2_sphere_2: origin xyz=0.0 -0.12 0.0 rpy=0.0 0.0 0.0 -> xyz=0.0 -0.12 0.0 rpy=0 0 0
- joint joint_panda_link2_sphere_3: origin xyz=0.0 -0.17 0.0 rpy=0.0 0.0 0.0 -> xyz=0.0 -0.17 0.0 rpy=0 0 0
- joint joint_panda_link3_sphere_0: origin xyz=0.0 0.0 -0.06 rpy=0.0 0.0 0.0 -> xyz=0.0 0.0 -0.06 rpy=0 0 0
- joint joint_panda_link3_sphere_1: origin xyz=0.0 0.0 -0.1 rpy=0.0 0.0 0.0 -> xyz=0.0 0.0 -0.1 rpy=0 0 0
- joint joint_panda_link3_sphere_2: origin xyz=0.08 0.06 0.0 rpy=0.0 0.0 0.0 -> xyz=0.08 0.06 0.0 rpy=0 0 0
- joint joint_panda_link3_sphere_3: origin xyz=0.08 0.02 0.0 rpy=0.0 0.0 0.0 -> xyz=0.08 0.02 0.0 rpy=0 0 0
- joint joint_panda_link4_sphere_0: origin xyz=0.0 0.0 0.02 rpy=0.0 0.0 0.0 -> xyz=0.0 0.0 0.02 rpy=0 0 0
- joint joint_panda_link4_sphere_1: origin xyz=0.0 0.0 0.06 rpy=0.0 0.0 0.0 -> xyz=0.0 0.0 0.06 rpy=0 0 0
- joint joint_panda_link4_sphere_2: origin xyz=-0.08 0.095 0.0 rpy=0.0 0.0 0.0 -> xyz=-0.08 0.095 0.0 rpy=0 0 0
- joint joint_panda_link4_sphere_3: origin xyz=-0.08 0.06 0.0 rpy=0.0 0.0 0.0 -> xyz=-0.08 0.06 0.0 rpy=0 0 0
- joint joint_panda_link5_sphere_0: origin xyz=0.0 0.055 0.0 rpy=0.0 0.0 0.0 -> xyz=0.0 0.055 0.0 rpy=0 0 0
- joint joint_panda_link5_sphere_1: origin xyz=0.0 0.075 0.0 rpy=0.0 0.0 0.0 -> xyz=0.0 0.075 0.0 rpy=0 0 0
- joint joint_panda_link5_sphere_10: origin xyz=-0.01 0.09 -0.08 rpy=0.0 0.0 0.0 -> xyz=-0.01 0.09 -0.08 rpy=0 0 0
- joint joint_panda_link5_sphere_11: origin xyz=-0.01 0.095 -0.05 rpy=0.0 0.0 0.0 -> xyz=-0.01 0.095 -0.05 rpy=0 0 0
- joint joint_panda_link5_sphere_2: origin xyz=0.0 0.0 -0.22 rpy=0.0 0.0 0.0 -> xyz=0.0 0.0 -0.22 rpy=0 0 0
- joint joint_panda_link5_sphere_3: origin xyz=0.0 0.05 -0.18 rpy=0.0 0.0 0.0 -> xyz=0.0 0.05 -0.18 rpy=0 0 0
- joint joint_panda_link5_sphere_4: origin xyz=0.01 0.08 -0.14 rpy=0.0 0.0 0.0 -> xyz=0.01 0.08 -0.14 rpy=0 0 0
- joint joint_panda_link5_sphere_5: origin xyz=0.01 0.085 -0.11 rpy=0.0 0.0 0.0 -> xyz=0.01 0.085 -0.11 rpy=0 0 0
- joint joint_panda_link5_sphere_6: origin xyz=0.01 0.09 -0.08 rpy=0.0 0.0 0.0 -> xyz=0.01 0.09 -0.08 rpy=0 0 0
- joint joint_panda_link5_sphere_7: origin xyz=0.01 0.095 -0.05 rpy=0.0 0.0 0.0 -> xyz=0.01 0.095 -0.05 rpy=0 0 0
- joint joint_panda_link5_sphere_8: origin xyz=-0.01 0.08 -0.14 rpy=0.0 0.0 0.0 -> xyz=-0.01 0.08 -0.14 rpy=0 0 0
- joint joint_panda_link5_sphere_9: origin xyz=-0.01 0.085 -0.11 rpy=0.0 0.0 0.0 -> xyz=-0.01 0.085 -0.11 rpy=0 0 0
- joint joint_panda_link6_sphere_0: origin xyz=0.0 0.0 0.0 rpy=0.0 0.0 0.0 -> xyz=0.0 0.0 0.0 rpy=0 0 0
- joint joint_panda_link6_sphere_1: origin xyz=0.08 0.03 0.0 rpy=0.0 0.0 0.0 -> xyz=0.08 0.03 0.0 rpy=0 0 0
- joint joint_panda_link6_sphere_2: origin xyz=0.08 -0.01 0.0 rpy=0.0 0.0 0.0 -> xyz=0.08 -0.01 0.0 rpy=0 0 0
- joint joint_panda_link7_sphere_0: origin xyz=0.0 0.0 0.07 rpy=0.0 0.0 0.0 -> xyz=0.0 0.0 0.07 rpy=0 0 0
- joint joint_panda_link7_sphere_1: origin xyz=0.02 0.04 0.08 rpy=0.0 0.0 0.0 -> xyz=0.02 0.04 0.08 rpy=0 0 0
- joint joint_panda_link7_sphere_2: origin xyz=0.04 0.02 0.08 rpy=0.0 0.0 0.0 -> xyz=0.04 0.02 0.08 rpy=0 0 0
- joint joint_panda_link7_sphere_3: origin xyz=0.04 0.06 0.085 rpy=0.0 0.0 0.0 -> xyz=0.04 0.06 0.085 rpy=0 0 0
- joint joint_panda_link7_sphere_4: origin xyz=0.06 0.04 0.085 rpy=0.0 0.0 0.0 -> xyz=0.06 0.04 0.085 rpy=0 0 0
