Commit message: Update isaac

File: torch_robotics/data/urdf/robots/franka_description/robots/panda_arm_hand_fixed_gripper_collision_model.urdf (robot description, URDF)
Before this commit: robot panda, 63 links, 62 joints
Links:
- link panda_hand_0: geometry visual sphere radius=0.028
- link panda_hand_1: geometry visual sphere radius=0.028
- link panda_hand_10: geometry visual sphere radius=0.026
- link panda_hand_11: geometry visual sphere radius=0.026
- link panda_hand_12: geometry visual sphere radius=0.024
- link panda_hand_13: geometry visual sphere radius=0.024
- link panda_hand_14: geometry visual sphere radius=0.024
- link panda_hand_15: geometry visual sphere radius=0.024
- link panda_hand_16: geometry visual sphere radius=0.024
- link panda_hand_17: geometry visual sphere radius=0.024
- link panda_hand_2: geometry visual sphere radius=0.028
- link panda_hand_3: geometry visual sphere radius=0.028
- link panda_hand_4: geometry visual sphere radius=0.028
- link panda_hand_5: geometry visual sphere radius=0.028
- link panda_hand_6: geometry visual sphere radius=0.026
- link panda_hand_7: geometry visual sphere radius=0.026
- link panda_hand_8: geometry visual sphere radius=0.026
- link panda_hand_9: geometry visual sphere radius=0.026
- link panda_link2_0: geometry visual sphere radius=0.06
- link panda_link2_1: geometry visual sphere radius=0.06
- link panda_link2_2: geometry visual sphere radius=0.06
- link panda_link2_3: geometry visual sphere radius=0.06
- link panda_link3_0: geometry visual sphere radius=0.05
- link panda_link3_1: geometry visual sphere radius=0.06
- link panda_link3_2: geometry visual sphere radius=0.055
- link panda_link3_3: geometry visual sphere radius=0.055
- link panda_link4_0: geometry visual sphere radius=0.055
- link panda_link4_1: geometry visual sphere radius=0.055
- link panda_link4_2: geometry visual sphere radius=0.06
- link panda_link4_3: geometry visual sphere radius=0.055
- link panda_link5_0: geometry visual sphere radius=0.06
- link panda_link5_1: geometry visual sphere radius=0.06
- link panda_link5_10: geometry visual sphere radius=0.025
- link panda_link5_11: geometry visual sphere radius=0.025
- link panda_link5_2: geometry visual sphere radius=0.06
- link panda_link5_3: geometry visual sphere radius=0.05
- link panda_link5_4: geometry visual sphere radius=0.025
- link panda_link5_5: geometry visual sphere radius=0.025
- link panda_link5_6: geometry visual sphere radius=0.025
- link panda_link5_7: geometry visual sphere radius=0.025
- link panda_link5_8: geometry visual sphere radius=0.025
- link panda_link5_9: geometry visual sphere radius=0.025
- link panda_link6_0: geometry visual sphere radius=0.06
- link panda_link6_1: geometry visual sphere radius=0.06
- link panda_link6_2: geometry visual sphere radius=0.06
- link panda_link7_0: geometry visual sphere radius=0.05
- link panda_link7_1: geometry visual sphere radius=0.025
- link panda_link7_2: geometry visual sphere radius=0.025
- link panda_link7_3: geometry visual sphere radius=0.02
- link panda_link7_4: geometry visual sphere radius=0.02

Commit message: Fix environment base

File: torch_robotics/data/urdf/robots/franka_description/robots/panda_arm_hand_fixed_gripper_collision_model.urdf (robot description, URDF)
Before this commit: robot panda, 63 links, 62 joints
Links:
- link panda_hand_0: geometry 
- link panda_hand_1: geometry 
- link panda_hand_10: geometry 
- link panda_hand_11: geometry 
- link panda_hand_12: geometry 
- link panda_hand_13: geometry 
- link panda_hand_14: geometry 
- link panda_hand_15: geometry 
- link panda_hand_16: geometry 
- link panda_hand_17: geometry 
- link panda_hand_2: geometry 
- link panda_hand_3: geometry 
- link panda_hand_4: geometry 
- link panda_hand_5: geometry 
- link panda_hand_6: geometry 
- link panda_hand_7: geometry 
- link panda_hand_8: geometry 
- link panda_hand_9: geometry 
- link panda_link2_0: geometry 
- link panda_link2_1: geometry 
- link panda_link2_2: geometry 
- link panda_link2_3: geometry 
- link panda_link3_0: geometry 
- link panda_link3_1: geometry 
- link panda_link3_2: geometry 
- link panda_link3_3: geometry 
- link panda_link4_0: geometry 
- link panda_link4_1: geometry 
- link panda_link4_2: geometry 
- link panda_link4_3: geometry 
- link panda_link5_0: geometry 
- link panda_link5_1: geometry 
- link panda_link5_10: geometry 
- link panda_link5_11: geometry 
- link panda_link5_2: geometry 
- link panda_link5_3: geometry 
- link panda_link5_4: geometry 
- link panda_link5_5: geometry 
- link panda_link5_6: geometry 
- link panda_link5_7: geometry 
- link panda_link5_8: geometry 
- link panda_link5_9: geometry 
- link panda_link6_0: geometry 
- link panda_link6_1: geometry 
- link panda_link6_2: geometry 
- link panda_link7_0: geometry 
- link panda_link7_1: geometry 
- link panda_link7_2: geometry 
- link panda_link7_3: geometry 
- link panda_link7_4: geometry 

Commit message: Fix collision spheres

File: torch_robotics/data/urdf/robots/franka_description/robots/panda_arm_hand_fixed_gripper_collision_model.urdf (robot description, URDF)
Before this commit: robot panda, 63 links, 62 joints
Links:
- added link panda_hand_18; visual sphere radius=0.02
- added link panda_hand_19; visual sphere radius=0.02
- added link panda_hand_20; visual sphere radius=0.02
- added link panda_hand_21; visual sphere radius=0.02
- added link panda_hand_22; visual sphere radius=0.02
- added link panda_hand_23; visual sphere radius=0.02
- link panda_hand_0: geometry visual sphere radius=0.028
- link panda_hand_1: geometry visual sphere radius=0.028
- link panda_hand_10: geometry visual sphere radius=0.026
- link panda_hand_11: geometry visual sphere radius=0.026
- link panda_hand_12: geometry visual sphere radius=0.024
- link panda_hand_13: geometry visual sphere radius=0.024
- link panda_hand_14: geometry visual sphere radius=0.024
- link panda_hand_15: geometry visual sphere radius=0.024
- link panda_hand_16: geometry visual sphere radius=0.024
- link panda_hand_17: geometry visual sphere radius=0.024
- link panda_hand_2: geometry visual sphere radius=0.028
- link panda_hand_3: geometry visual sphere radius=0.028
- link panda_hand_4: geometry visual sphere radius=0.028
- link panda_hand_5: geometry visual sphere radius=0.028
- link panda_hand_6: geometry visual sphere radius=0.026
- link panda_hand_7: geometry visual sphere radius=0.026
- link panda_hand_8: geometry visual sphere radius=0.026
- link panda_hand_9: geometry visual sphere radius=0.026
- link panda_link2_0: geometry visual sphere radius=0.06
- link panda_link2_1: geometry visual sphere radius=0.06
- link panda_link2_2: geometry visual sphere radius=0.06
- link panda_link2_3: geometry visual sphere radius=0.06
- link panda_link3_0: geometry visual sphere radius=0.05
- link panda_link3_1: geometry visual sphere radius=0.06
- link panda_link3_2: geometry visual sphere radius=0.055
- link panda_link3_3: geometry visual sphere radius=0.055
- link panda_link4_0: geometry visual sphere radius=0.055
- link panda_link4_1: geometry visual sphere radius=0.055
- link panda_link4_2: geometry visual sphere radius=0.06
- link panda_link4_3: geometry visual sphere radius=0.055
- link panda_link5_0: geometry visual sphere radius=0.06
- link panda_link5_1: geometry visual sphere radius=0.06
- link panda_link5_10: geometry visual sphere radius=0.025
- link panda_link5_11: geometry visual sphere radius=0.025
- link panda_link5_2: geometry visual sphere radius=0.06
- link panda_link5_3: geometry visual sphere radius=0.05
- link panda_link5_4: geometry visual sphere radius=0.025
- link panda_link5_5: geometry visual sphere radius=0.025
- link panda_link5_6: geometry visual sphere radius=0.025
- link panda_link5_7: geometry visual sphere radius=0.025
- link panda_link5_8: geometry visual sphere radius=0.025
- link panda_link5_9: geometry visual sphere radius=0.025
- link panda_link6_0: geometry visual sphere radius=0.06
- link panda_link6_1: geometry visual sphere radius=0.06
- link panda_link6_2: geometry visual sphere radius=0.06
- link panda_link7_0: geometry visual sphere radius=0.05
- link panda_link7_1: geometry visual sphere radius=0.025
- link panda_link7_2: geometry visual sphere radius=0.025
- link panda_link7_3: geometry visual sphere radius=0.02
- link panda_link7_4: geometry visual sphere radius=0.02
Joints:
- added joint joint_panda_hand_sphere_18: type fixed, parent panda_hand, child panda_hand_18, origin xyz=0.0 -0.075 0.08 rpy=0 0 0
- added joint joint_panda_hand_sphere_19: type fixed, parent panda_hand, child panda_hand_19, origin xyz=0.0 -0.045 0.08 rpy=0 0 0
- added joint joint_panda_hand_sphere_20: type fixed, parent panda_hand, child panda_hand_20, origin xyz=0.0 -0.015 0.08 rpy=0 0 0
- added joint joint_panda_hand_sphere_21: type fixed, parent panda_hand, child panda_hand_21, origin xyz=0.0 0.015 0.08 rpy=0 0 0
- added joint joint_panda_hand_sphere_22: type fixed, parent panda_hand, child panda_hand_22, origin xyz=0.0 0.045 0.08 rpy=0 0 0
- added joint joint_panda_hand_sphere_23: type fixed, parent panda_hand, child panda_hand_23, origin xyz=0.0 0.075 0.08 rpy=0 0 0

File: torch_robotics/data/urdf/robots/franka_description/robots/panda_arm_hand_no_gripper_collision_model.urdf (robot description, URDF)
Before this commit: robot panda, 61 links, 60 joints
Links:
- added link panda_hand_18; visual sphere radius=0.02
- added link panda_hand_19; visual sphere radius=0.02
- added link panda_hand_20; visual sphere radius=0.02
- added link panda_hand_21; visual sphere radius=0.02
- added link panda_hand_22; visual sphere radius=0.02
- added link panda_hand_23; visual sphere radius=0.02
- link panda_hand_0: geometry visual sphere radius=0.028
- link panda_hand_1: geometry visual sphere radius=0.028
- link panda_hand_10: geometry visual sphere radius=0.026
- link panda_hand_11: geometry visual sphere radius=0.026
- link panda_hand_12: geometry visual sphere radius=0.024
- link panda_hand_13: geometry visual sphere radius=0.024
- link panda_hand_14: geometry visual sphere radius=0.024
- link panda_hand_15: geometry visual sphere radius=0.024
- link panda_hand_16: geometry visual sphere radius=0.024
- link panda_hand_17: geometry visual sphere radius=0.024
- link panda_hand_2: geometry visual sphere radius=0.028
- link panda_hand_3: geometry visual sphere radius=0.028
- link panda_hand_4: geometry visual sphere radius=0.028
- link panda_hand_5: geometry visual sphere radius=0.028
- link panda_hand_6: geometry visual sphere radius=0.026
- link panda_hand_7: geometry visual sphere radius=0.026
- link panda_hand_8: geometry visual sphere radius=0.026
- link panda_hand_9: geometry visual sphere radius=0.026
- link panda_link2_0: geometry visual sphere radius=0.06
- link panda_link2_1: geometry visual sphere radius=0.06
- link panda_link2_2: geometry visual sphere radius=0.06
- link panda_link2_3: geometry visual sphere radius=0.06
- link panda_link3_0: geometry visual sphere radius=0.05
- link panda_link3_1: geometry visual sphere radius=0.06
- link panda_link3_2: geometry visual sphere radius=0.055
- link panda_link3_3: geometry visual sphere radius=0.055
- link panda_link4_0: geometry visual sphere radius=0.055
- link panda_link4_1: geometry visual sphere radius=0.055
- link panda_link4_2: geometry visual sphere radius=0.06
- link panda_link4_3: geometry visual sphere radius=0.055
- link panda_link5_0: geometry visual sphere radius=0.06
- link panda_link5_1: geometry visual sphere radius=0.06
- link panda_link5_10: geometry visual sphere radius=0.025
- link panda_link5_11: geometry visual sphere radius=0.025
- link panda_link5_2: geometry visual sphere radius=0.06
- link panda_link5_3: geometry visual sphere radius=0.05
- link panda_link5_4: geometry visual sphere radius=0.025
- link panda_link5_5: geometry visual sphere radius=0.025
- link panda_link5_6: geometry visual sphere radius=0.025
- link panda_link5_7: geometry visual sphere radius=0.025
- link panda_link5_8: geometry visual sphere radius=0.025
- link panda_link5_9: geometry visual sphere radius=0.025
- link panda_link6_0: geometry visual sphere radius=0.06
- link panda_link6_1: geometry visual sphere radius=0.06
- link panda_link6_2: geometry visual sphere radius=0.06
- link panda_link7_0: geometry visual sphere radius=0.05
- link panda_link7_1: geometry visual sphere radius=0.025
- link panda_link7_2: geometry visual sphere radius=0.025
- link panda_link7_3: geometry visual sphere radius=0.02
- link panda_link7_4: geometry visual sphere radius=0.02
Joints:
- added joint joint_panda_hand_sphere_18: type fixed, parent panda_hand, child panda_hand_18, origin xyz=0.0 -0.075 0.08 rpy=0 0 0
- added joint joint_panda_hand_sphere_19: type fixed, parent panda_hand, child panda_hand_19, origin xyz=0.0 -0.045 0.08 rpy=0 0 0
- added joint joint_panda_hand_sphere_20: type fixed, parent panda_hand, child panda_hand_20, origin xyz=0.0 -0.015 0.08 rpy=0 0 0
- added joint joint_panda_hand_sphere_21: type fixed, parent panda_hand, child panda_hand_21, origin xyz=0.0 0.015 0.08 rpy=0 0 0
- added joint joint_panda_hand_sphere_22: type fixed, parent panda_hand, child panda_hand_22, origin xyz=0.0 0.045 0.08 rpy=0 0 0
- added joint joint_panda_hand_sphere_23: type fixed, parent panda_hand, child panda_hand_23, origin xyz=0.0 0.075 0.08 rpy=0 0 0

File: torch_robotics/data/urdf/robots/planar_robot/planar_robot_2_link.urdf (robot description, URDF)
Before this commit: robot planar_robot_2_link, 5 links, 4 joints
Links:
- link link_2: geometry collision cylinder length=0.3 radius=0.01; visual cylinder length=0.3 radius=0.01
Joints:
- joint joint_1: limit lower=-2.9670597283903604 upper=2.9670597283903604 effort=320.0 velocity=2.35619449019 -> lower=-2.97 upper=2.97 effort=320.0 velocity=2.35619449019
- joint joint_2: limit lower=-2.0943951023931953 upper=2.0943951023931953 effort=320.0 velocity=2.35619449019 -> lower=-2.6 upper=2.6 effort=320.0 velocity=2.35619449019
- joint joint_ee: origin xyz=0.4 0 0.0 -> xyz=0.3 0 0.0

File: torch_robotics/data/urdf/robots/planar_robot/planar_robot_4_link_collision_model.urdf (robot description, URDF)
Before this commit: robot planar_robot_4_link, 28 links, 27 joints
Links:
- link link_1_0: geometry visual sphere radius=0.01
- link link_1_1: geometry visual sphere radius=0.01
- link link_1_2: geometry visual sphere radius=0.01
- link link_1_3: geometry visual sphere radius=0.01
- link link_1_4: geometry visual sphere radius=0.01
- link link_2_0: geometry visual sphere radius=0.01
- link link_2_1: geometry visual sphere radius=0.01
- link link_2_2: geometry visual sphere radius=0.01
- link link_2_3: geometry visual sphere radius=0.01
- link link_2_4: geometry visual sphere radius=0.01
- link link_3_0: geometry visual sphere radius=0.01
- link link_3_1: geometry visual sphere radius=0.01
- link link_3_2: geometry visual sphere radius=0.01
- link link_3_3: geometry visual sphere radius=0.01
- link link_3_4: geometry visual sphere radius=0.01
- link link_4_0: geometry visual sphere radius=0.01
- link link_4_1: geometry visual sphere radius=0.01
- link link_4_2: geometry visual sphere radius=0.01
- link link_4_3: geometry visual sphere radius=0.01
- link link_4_4: geometry visual sphere radius=0.01
- link link_4_5: geometry visual sphere radius=0.02

Commit message: Panda spheres grippers

File: torch_robotics/data/urdf/robots/franka_description/robots/panda_arm_hand_fixed_gripper_collision_model.urdf (robot description, URDF)
Before this commit: robot panda, 69 links, 68 joints
Links:
- removed link panda_hand_20
- removed link panda_hand_21
- removed link panda_hand_22
- removed link panda_hand_23
- link panda_hand_0: geometry 
- link panda_hand_1: geometry 
- link panda_hand_10: geometry 
- link panda_hand_11: geometry 
- link panda_hand_12: geometry 
- link panda_hand_13: geometry 
- link panda_hand_14: geometry 
- link panda_hand_15: geometry 
- link panda_hand_16: geometry 
- link panda_hand_17: geometry 
- link panda_hand_18: geometry 
- link panda_hand_19: geometry 
- link panda_hand_2: geometry 
- link panda_hand_3: geometry 
- link panda_hand_4: geometry 
- link panda_hand_5: geometry 
- link panda_hand_6: geometry 
- link panda_hand_7: geometry 
- link panda_hand_8: geometry 
- link panda_hand_9: geometry 
- link panda_link2_0: geometry 
- link panda_link2_1: geometry 
- link panda_link2_2: geometry 
- link panda_link2_3: geometry 
- link panda_link3_0: geometry 
- link panda_link3_1: geometry 
- link panda_link3_2: geometry 
- link panda_link3_3: geometry 
- link panda_link4_0: geometry 
- link panda_link4_1: geometry 
- link panda_link4_2: geometry 
- link panda_link4_3: geometry 
- link panda_link5_0: geometry 
- link panda_link5_1: geometry 
- link panda_link5_10: geometry 
- link panda_link5_11: geometry 
- link panda_link5_2: geometry 
- link panda_link5_3: geometry 
- link panda_link5_4: geometry 
- link panda_link5_5: geometry 
- link panda_link5_6: geometry 
- link panda_link5_7: geometry 
- link panda_link5_8: geometry 
- link panda_link5_9: geometry 
- link panda_link6_0: geometry 
- link panda_link6_1: geometry 
- link panda_link6_2: geometry 
- link panda_link7_0: geometry 
- link panda_link7_1: geometry 
- link panda_link7_2: geometry 
- link panda_link7_3: geometry 
- link panda_link7_4: geometry 
Joints:
- removed joint joint_panda_hand_sphere_20
- removed joint joint_panda_hand_sphere_21
- removed joint joint_panda_hand_sphere_22
- removed joint joint_panda_hand_sphere_23
- joint joint_panda_hand_sphere_18: origin xyz=0.0 -0.075 0.08 rpy=0 0 0 -> xyz=0.0 -0.045 0.085 rpy=0 0 0
- joint joint_panda_hand_sphere_19: origin xyz=0.0 -0.045 0.08 rpy=0 0 0 -> xyz=0.0 0.045 0.085 rpy=0 0 0

File: torch_robotics/data/urdf/robots/franka_description/robots/panda_arm_hand_no_gripper_collision_model.urdf (robot description, URDF)
Before this commit: robot panda, 67 links, 66 joints
Links:
- removed link panda_hand_20
- removed link panda_hand_21
- removed link panda_hand_22
- removed link panda_hand_23
- link panda_hand_0: geometry 
- link panda_hand_1: geometry 
- link panda_hand_10: geometry 
- link panda_hand_11: geometry 
- link panda_hand_12: geometry 
- link panda_hand_13: geometry 
- link panda_hand_14: geometry 
- link panda_hand_15: geometry 
- link panda_hand_16: geometry 
- link panda_hand_17: geometry 
- link panda_hand_18: geometry 
- link panda_hand_19: geometry 
- link panda_hand_2: geometry 
- link panda_hand_3: geometry 
- link panda_hand_4: geometry 
- link panda_hand_5: geometry 
- link panda_hand_6: geometry 
- link panda_hand_7: geometry 
- link panda_hand_8: geometry 
- link panda_hand_9: geometry 
- link panda_link2_0: geometry 
- link panda_link2_1: geometry 
- link panda_link2_2: geometry 
- link panda_link2_3: geometry 
- link panda_link3_0: geometry 
- link panda_link3_1: geometry 
- link panda_link3_2: geometry 
- link panda_link3_3: geometry 
- link panda_link4_0: geometry 
- link panda_link4_1: geometry 
- link panda_link4_2: geometry 
- link panda_link4_3: geometry 
- link panda_link5_0: geometry 
- link panda_link5_1: geometry 
- link panda_link5_10: geometry 
- link panda_link5_11: geometry 
- link panda_link5_2: geometry 
- link panda_link5_3: geometry 
- link panda_link5_4: geometry 
- link panda_link5_5: geometry 
- link panda_link5_6: geometry 
- link panda_link5_7: geometry 
- link panda_link5_8: geometry 
- link panda_link5_9: geometry 
- link panda_link6_0: geometry 
- link panda_link6_1: geometry 
- link panda_link6_2: geometry 
- link panda_link7_0: geometry 
- link panda_link7_1: geometry 
- link panda_link7_2: geometry 
- link panda_link7_3: geometry 
- link panda_link7_4: geometry 
Joints:
- removed joint joint_panda_hand_sphere_20
- removed joint joint_panda_hand_sphere_21
- removed joint joint_panda_hand_sphere_22
- removed joint joint_panda_hand_sphere_23
- joint joint_panda_hand_sphere_18: origin xyz=0.0 -0.075 0.08 rpy=0 0 0 -> xyz=0.0 -0.045 0.085 rpy=0 0 0
- joint joint_panda_hand_sphere_19: origin xyz=0.0 -0.045 0.08 rpy=0 0 0 -> xyz=0.0 0.045 0.085 rpy=0 0 0

File: torch_robotics/data/urdf/robots/planar_robot/planar_robot_4_link_collision_model.urdf (robot description, URDF)
Before this commit: robot planar_robot_4_link, 28 links, 27 joints
Links:
- link link_1_0: geometry 
- link link_1_1: geometry 
- link link_1_2: geometry 
- link link_1_3: geometry 
- link link_1_4: geometry 
- link link_2_0: geometry 
- link link_2_1: geometry 
- link link_2_2: geometry 
- link link_2_3: geometry 
- link link_2_4: geometry 
- link link_3_0: geometry 
- link link_3_1: geometry 
- link link_3_2: geometry 
- link link_3_3: geometry 
- link link_3_4: geometry 
- link link_4_0: geometry 
- link link_4_1: geometry 
- link link_4_2: geometry 
- link link_4_3: geometry 
- link link_4_4: geometry 
- link link_4_5: geometry 
