Commit message: Add 4 link robot

File: torch_robotics/data/urdf/robots/planar_robot_4_link.urdf (robot description, URDF)
Before this commit: robot planar_robot_2_link, 5 links, 4 joints
Links:
- added link link_3; collision cylinder length=0.2 radius=0.01; visual cylinder length=0.2 radius=0.01
- added link link_4; collision cylinder length=0.2 radius=0.01; visual cylinder length=0.2 radius=0.01
- link link_2: geometry collision cylinder length=0.2 radius=0.01; visual cylinder length=0.2 radius=0.01
Joints:
- added joint joint_3: type revolute, parent link_2, child link_3, origin xyz=0.2 0 0, axis 0 0 1, limit lower=-2.36 upper=2.36 effort=320.0 velocity=2.35619449019
- added joint joint_4: type revolute, parent link_3, child link_4, origin xyz=0.2 0 0, axis 0 0 1, limit lower=-2.36 upper=2.36 effort=320.0 velocity=2.35619449019
- joint joint_1: limit lower=-2.9670597283903604 upper=2.9670597283903604 effort=320.0 velocity=2.35619449019 -> lower=-2.97 upper=2.97 effort=320.0 velocity=2.35619449019
- joint joint_2: limit lower=-2.0943951023931953 upper=2.0943951023931953 effort=320.0 velocity=2.35619449019 -> lower=-2.36 upper=2.36 effort=320.0 velocity=2.35619449019
- joint joint_ee: origin xyz=0.4 0 0.0 -> xyz=0.2 0 0.0; parent link_2 -> link_4

File: torch_robotics/data/urdf/robots/planar_robot_4_link_collision_model.urdf (robot description, URDF)
Before this commit: robot planar_robot_2_link, 19 links, 18 joints
Links:
- removed link link_2_5
- removed link link_2_6
- removed link link_2_7
- removed link link_2_8
- added link link_3; collision cylinder length=0.2 radius=0.01; visual cylinder length=0.2 radius=0.01
- added link link_3_0; visual sphere radius=0.01
- added link link_3_1; visual sphere radius=0.01
- added link link_3_2; visual sphere radius=0.01
- added link link_3_3; visual sphere radius=0.01
- added link link_3_4; visual sphere radius=0.01
- added link link_4; collision cylinder length=0.2 radius=0.01; visual cylinder length=0.2 radius=0.01
- added link link_4_0; visual sphere radius=0.01
- added link link_4_1; visual sphere radius=0.01
- added link link_4_2; visual sphere radius=0.01
- added link link_4_3; visual sphere radius=0.01
- added link link_4_4; visual sphere radius=0.01
- added link link_4_5; visual sphere radius=0.01
- link link_2: geometry collision cylinder length=0.2 radius=0.01; visual cylinder length=0.2 radius=0.01
Joints:
- removed joint joint_link_2_sphere_5
- removed joint joint_link_2_sphere_6
- removed joint joint_link_2_sphere_7
- removed joint joint_link_2_sphere_8
- added joint joint_3: type revolute, parent link_2, child link_3, origin xyz=0.2 0.0 0.0 rpy=0 0 0, axis 0.0 0.0 1.0, limit lower=-2.36 upper=2.36 effort=320.0 velocity=2.35619449019
- added joint joint_4: type revolute, parent link_3, child link_4, origin xyz=0.2 0.0 0.0 rpy=0 0 0, axis 0.0 0.0 1.0, limit lower=-2.36 upper=2.36 effort=320.0 velocity=2.35619449019
- added joint joint_link_3_sphere_0: type fixed, parent link_3, child link_3_0, origin xyz=0.0 0.0 0.0 rpy=0 0 0
- added joint joint_link_3_sphere_1: type fixed, parent link_3, child link_3_1, origin xyz=0.04 0.0 0.0 rpy=0 0 0
- added joint joint_link_3_sphere_2: type fixed, parent link_3, child link_3_2, origin xyz=0.08 0.0 0.0 rpy=0 0 0
- added joint joint_link_3_sphere_3: type fixed, parent link_3, child link_3_3, origin xyz=0.12 0.0 0.0 rpy=0 0 0
- added joint joint_link_3_sphere_4: type fixed, parent link_3, child link_3_4, origin xyz=0.16 0.0 0.0 rpy=0 0 0
- added joint joint_link_4_sphere_0: type fixed, parent link_4, child link_4_0, origin xyz=0.0 0.0 0.0 rpy=0 0 0
- added joint joint_link_4_sphere_1: type fixed, parent link_4, child link_4_1, origin xyz=0.04 0.0 0.0 rpy=0 0 0
- added joint joint_link_4_sphere_2: type fixed, parent link_4, child link_4_2, origin xyz=0.08 0.0 0.0 rpy=0 0 0
- added joint joint_link_4_sphere_3: type fixed, parent link_4, child link_4_3, origin xyz=0.12 0.0 0.0 rpy=0 0 0
- added joint joint_link_4_sphere_4: type fixed, parent link_4, child link_4_4, origin xyz=0.16 0.0 0.0 rpy=0 0 0
- added joint joint_link_4_sphere_5: type fixed, parent link_4, child link_4_5, origin xyz=0.2 0.0 0.0 rpy=0 0 0
- joint joint_1: limit lower=-2.9670597283903604 upper=2.9670597283903604 effort=320.0 velocity=2.35619449019 -> lower=-2.97 upper=2.97 effort=320.0 velocity=2.35619449019
- joint joint_2: limit lower=-2.0943951023931953 upper=2.0943951023931953 effort=320.0 velocity=2.35619449019 -> lower=-2.36 upper=2.36 effort=320.0 velocity=2.35619449019
- joint joint_ee: origin xyz=0.4 0.0 0.0 rpy=0 0 0 -> xyz=0.2 0.0 0.0 rpy=0 0 0; parent link_2 -> link_4
- joint joint_link_2_sphere_1: origin xyz=0.05 0.0 0.0 rpy=0 0 0 -> xyz=0.04 0.0 0.0 rpy=0 0 0
- joint joint_link_2_sphere_2: origin xyz=0.1 0.0 0.0 rpy=0 0 0 -> xyz=0.08 0.0 0.0 rpy=0 0 0
- joint joint_link_2_sphere_3: origin xyz=0.15 0.0 0.0 rpy=0 0 0 -> xyz=0.12 0.0 0.0 rpy=0 0 0
- joint joint_link_2_sphere_4: origin xyz=0.2 0.0 0.0 rpy=0 0 0 -> xyz=0.16 0.0 0.0 rpy=0 0 0
