Commit message: Collision models urdf

File: torch_robotics/data/urdf/robots/planar_robot_2_link_collision_model.urdf (robot description, URDF)
Before this commit: robot planar_robot_2_link, 19 links, 18 joints
Links:
- link link_1_0: geometry 
- link link_1_1: geometry 
- link link_1_2: geometry 
- link link_1_3: geometry 
- link link_1_4: geometry 
- link link_2_0: geometry 
- link link_2_1: geometry 
- link link_2_2: geometry 
- link link_2_3: geometry 
- link link_2_4: geometry 
- link link_2_5: geometry 
- link link_2_6: geometry 
- link link_2_7: geometry 
- link link_2_8: geometry 

File: torch_robotics/data/urdf/robots/planar_robot_4_link_collision_model.urdf (robot description, URDF)
Before this commit: robot planar_robot_4_link, 28 links, 27 joints
Links:
- link link_1_0: geometry 
- link link_1_1: geometry 
- link link_1_2: geometry 
- link link_1_3: geometry 
- link link_1_4: geometry 
- link link_2_0: geometry 
- link link_2_1: geometry 
- link link_2_2: geometry 
- link link_2_3: geometry 
- link link_2_4: geometry 
- link link_3_0: geometry 
- link link_3_1: geometry 
- link link_3_2: geometry 
- link link_3_3: geometry 
- link link_3_4: geometry 
- link link_4_0: geometry 
- link link_4_1: geometry 
- link link_4_2: geometry 
- link link_4_3: geometry 
- link link_4_4: geometry 
- link link_4_5: geometry 
